File: PCB/E32CB_R2/chamber-board.sch (KiCad schematic (older format))
At the start: 89 parts, among them J1 HEADER_2x10_PARALLEL, J10 S, J11 D, J12 S, J13 D, J14 S, J15 D, J16 S, J17 D, J18 S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

Commit message: renamed board
Parts:
- J3: symbol E32CB_R2-rescue:USB_B-Connector -> chamber-board-rescue:USB_B-Connector-E32CB_R2-rescue
Changed lines of the file:
@@
 $EndDescr
 $Comp
-L E32CB_R2-rescue:USB_B-Connector J3
+L chamber-board-rescue:USB_B-Connector-E32CB_R2-rescue J3
 U 1 1 5DA1F910
 P 1350 1200
